File: BikeCam.kicad_pcb (KiCad board)
At the start: 2 copper layers, 23 parts, among them IC1 FS312F-G, J1 USB_OTG, J2 Conn_01x02_Female, Q1 IRLZ34N, Q2 IRLZ34N, Q3 IRLML5203, Q4 IRLML5203, U1 MCP73831-2-OT, U2 LTC3531ES6-3_3

Commit message: pcb trace
Parts:
- removed IC1: FS312F-G, Package_TO_SOT_SMD:SOT-23-6
- removed L1: 10uH, Inductor_SMD:L_1812_4532Metric
- added J3: Conn_01x02_Male, Connector_PinHeader_1.00mm:PinHeader_1x02_P1.00mm_Vertical, F.Cu at (94.0, 81.9)
- added SW1: SW_DIP_x01, Connector_PinHeader_1.00mm:PinHeader_1x02_P1.00mm_Vertical, F.Cu at (154.9, 57.1)
- added U3: MCP1700-3302E_SOT23, Package_TO_SOT_SMD:SOT-23, F.Cu at (180.3, 66.0)
- C4: value 2.2uF -> 1uF
- C5: value 10uF -> 1uF
- R3: value 1k -> 2.7k
- U2: value LTC3531ES6-3_3 -> AP9101CK6; footprint Package_TO_SOT_SMD:TSOT-23-6 -> Package_TO_SOT_SMD:SOT-23-6
- moved R1 78.4 mm to (89.5, 80.3), turned to 90 degrees
- moved C1 77.5 mm to (93.3, 75.6), turned to 90 degrees
- moved R3 66.1 mm to (97.8, 78.7)
- moved U2 62.9 mm to (116.2, 76.2), turned to -90 degrees
- moved U1 49.6 mm to (90.2, 76.2), turned to 180 degrees
- moved R2 46.6 mm to (95.2, 75.6), turned to -90 degrees
- moved R5 37.4 mm to (139.1, 64.8)
- moved C3 33.5 mm to (141.1, 78.1)
- moved R4 32.7 mm to (115.6, 81.3), turned to -90 degrees
- moved D2 32.4 mm to (153.0, 68.6), turned to 0 degrees
- moved J1 31.4 mm to (84.5, 76.8)
- moved Q1 30.1 mm to (130.0, 85.7), turned to 0 degrees
- moved Q2 29.3 mm to (125.1, 85.7), turned to 0 degrees
- moved C2 28.9 mm to (120.7, 77.0)
- moved C4 28.6 mm to (165.8, 80.3)
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Connections:
- C3 pad 2: OUT+ -> Net-(C3-Pad2)
- D2 pad 1: OUT+ -> Net-(C3-Pad2)
- Q1 pad 1: Net-(IC1-Pad3) -> Net-(Q1-Pad1)
- Q2 pad 1: Net-(IC1-Pad1) -> Net-(Q2-Pad1)
- Q4 pad 3: OUT+ -> Net-(C3-Pad2)
- R3 pad 1: Net-(IC1-Pad2) -> Net-(R3-Pad1)
- U2 pad 1: Net-(L1-Pad2) -> Net-(Q2-Pad1)
- U2 pad 2: 0V -> Net-(R3-Pad1)
- U2 pad 3: +3.3V -> Net-(Q1-Pad1)
- U2 pad 4: OUT+ -> unconnected-(U2-Pad4)
- U2 pad 5: OUT+ -> Net-(C2-Pad2)
- U2 pad 6: Net-(L1-Pad1) -> LIPO-
Routing:
- net +5V: track 0.00 -> 7.09 mm
- net Net-(D1-Pad1): track 0.00 -> 4.71 mm
- net Net-(R2-Pad2): track 0.00 -> 4.18 mm
- net LIPO+: track 0.00 -> 2.11 mm
- net 0V: track 0.00 -> 2.10 mm

Commit message: pwr module debugging
Parts:
- C2, Q1, Q2, R3, R4, U2: moved to B.Cu
- moved J2 77.3 mm to (114.7, 91.7), turned to 180 degrees
- moved U3 76.0 mm to (108.1, 89.7), turned to 180 degrees
- moved C5 62.0 mm to (113.2, 91.2), turned to -90 degrees
- moved C4 58.9 mm to (108.0, 92.2)
- moved SW1 56.4 mm to (111.1, 92.7), turned to -90 degrees
- moved R5 45.0 mm to (97.9, 83.1), turned to 180 degrees
- moved R6 44.7 mm to (105.5, 83.1), turned to 180 degrees
- moved D2 43.6 mm to (111.7, 82.5), turned to 180 degrees
- moved Q4 37.8 mm to (112.1, 86.2), turned to 0 degrees
- moved Q3 37.5 mm to (107.9, 86.2), turned to 0 degrees
- moved Q1 32.1 mm to (98.6, 92.1), turned to 180 degrees
- moved C3 30.4 mm to (112.7, 89.0), turned to 90 degrees
- moved Q2 23.0 mm to (103.0, 92.1), turned to 180 degrees
- moved C2 20.4 mm to (102.0, 85.1), turned to 180 degrees
- moved U2 19.3 mm to (101.1, 88.2), turned to 90 degrees
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Routing:
- net LIPO-: track 0.00 -> 25.4 mm, vias 0 -> 1
- net LIPO+: track 2.11 -> 24.4 mm
- net +5V: track 7.09 -> 25.1 mm
- net 0V: track 2.10 -> 18.1 mm, vias 0 -> 5
- net Net-(C3-Pad2): track 0.00 -> 11.8 mm
- net Net-(Q3-Pad1): track 0.00 -> 6.53 mm
- net Net-(C2-Pad2): track 0.00 -> 5.74 mm
- net OUT+: track 0.00 -> 4.91 mm
- net Net-(Q1-Pad2): track 0.00 -> 4.44 mm
- net Net-(Q3-Pad2): track 0.00 -> 4.19 mm
- net Net-(R3-Pad1): track 0.00 -> 3.93 mm
- net +3.3V: track 0.00 -> 3.15 mm, vias 0 -> 1
- net Net-(R1-Pad2): track 0.00 -> 2.85 mm
- net Net-(Q2-Pad1): track 0.00 -> 2.61 mm
- net Net-(Q1-Pad1): track 0.00 -> 1.99 mm
- added copper zone on In2.Cu, net +3.3V
- added copper zone on In1.Cu, net 0V
Other:
- board outline added: 25.4 x 14.7 mm
- copper layers 2 -> 4

Commit message: v1
Parts:
- J2: footprint Connector_PinSocket_1.00mm:PinSocket_1x02_P1.00mm_Vertical -> Connector_PinSocket_2.00mm:PinSocket_1x02_P2.00mm_Vertical
- J3, SW1: footprint Connector_PinHeader_1.00mm:PinHeader_1x02_P1.00mm_Vertical -> Connector_PinHeader_2.00mm:PinHeader_1x02_P2.00mm_Vertical
- moved J3 2.93 mm to (99.6, 82.3), turned to 90 degrees
- moved R5 1.89 mm to (96.0, 83.1)
- moved C4 1.67 mm to (106.4, 91.9)
- moved J2 0.64 mm to (115.3, 91.7)
- moved SW1 0.25 mm to (111.1, 93.0)
Connections:
- J3 pad 1: LIPO- -> LIPO+
- J3 pad 2: LIPO+ -> LIPO-
Routing:
- net 0V: track 18.1 -> 23.2 mm, vias 5 -> 4
- net +5V: track 25.1 -> 28.4 mm
- net LIPO+: track 24.4 -> 22.8 mm
- net LIPO-: track 25.4 -> 26.3 mm, vias 1 -> 0
- net +3.3V: track 3.15 -> 3.79 mm
Other:
- board size 25.4 x 14.7 mm -> 26.4 x 16.3 mm

Commit message: error debug
Connections:
- net +3.3V renamed +3V3
Routing:
- net unconnected-(J1-Pad6): track 0.00 -> 12.6 mm
Changed lines of the file:
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@@
   (net 4 "Net-(C2-Pad2)")
   (net 5 "OUT+")
-  (net 6 "+3.3V")
+  (net 6 "+3V3")
   (net 7 "Net-(D1-Pad1)")
   (net 8 "+5V")
@@
       (net 1 "0V") (pinfunction "GND") (pintype "power_in"))
     (pad "2" smd roundrect (at -0.9375 0.95 180) (size 1.475 0.6) (layers "F.Cu" "F.Paste" "F.Mask") (roundrect_rratio 0.25)
-      (net 6 "+3.3V") (pinfunction "VO") (pintype "power_out"))
+      (net 6 "+3V3") (pinfunction "VO") (pintype "power_out"))
     (pad "3" smd roundrect (at 0.9375 0 180) (size 1.475 0.6) (layers "F.Cu" "F.Paste" "F.Mask") (roundrect_rratio 0.25)
       (net 5 "OUT+") (pinfunction "VI") (pintype "power_in"))
@@
       (net 1 "0V") (pintype "passive"))
     (pad "2" smd roundrect (at 0.48 0 270) (size 0.56 0.62) (layers "F.Cu" "F.Paste" "F.Mask") (roundrect_rratio 0.25)
-      (net 6 "+3.3V") (pintype "passive"))
+      (net 6 "+3V3") (pintype "passive"))
     (model "${KICAD6_3DMODEL_DIR}/Capacitor_SMD.3dshapes/C_0402_1005Metric.wrl"
       (offset (xyz 0 0 0))
@@
     (fp_line (start -1 -1) (end 0.5 -1) (layer "F.Fab") (width 0.1))
     (pad "1" thru_hole rect (at 0 0 180) (size 1.35 1.35) (drill 0.8) (layers *.Cu *.Mask)
-      (net 6 "+3.3V") (pinfunction "Pin_1") (pintype "passive"))
+      (net 6 "+3V3") (pinfunction "Pin_1") (pintype "passive"))
     (pad "2" thru_hole oval (at 0 2 180) (size 1.35 1.35) (drill 0.8) (layers *.Cu *.Mask)
       (net 1 "0V") (pinfunction "Pin_2") (pintype "passive"))
@@
   (segment (start 108.048767 81.450001) (end 106.128999 81.450001) (width 0.6) (layer "F.Cu") (net 8))
   (segment (start 102.368 81.434299) (end 103.991701 83.058) (width 0.6) (layer "F.Cu") (net 8))
+  (segment (start 92.272 91.422) (end 93.467 92.617) (width 0.25) (layer "F.Cu") (net 12))
+  (segment (start 93.467 87.977) (end 94.502 87.977) (width 0.25) (layer "F.Cu") (net 12))
+  (segment (start 92.272 86.722) (end 92.272 89.172) (width 0.25) (layer "F.Cu") (net 12))
+  (segment (start 92.272 91.422) (end 92.272 93.872) (width 0.25) (layer "F.Cu") (net 12))
+  (segment (start 93.467 92.617) (end 94.502 92.617) (width 0.25) (layer "F.Cu") (net 12))
+  (segment (start 92.272 89.172) (end 93.467 87.977) (width 0.25) (layer "F.Cu") (net 12))
+  (segment (start 92.272 89.172) (end 92.272 91.422) (width 0.25) (layer "F.Cu") (net 12))
   (segment (start 99.4895 93.00825) (end 103.9345 93.00825) (width 0.47) (layer "B.Cu") (net 13))
   (segment (start 106.521 84.809) (end 106.934 85.222) (width 0.6) (layer "F.Cu") (net 14))
@@
     )
   )
-  (zone (net 6) (net_name "+3.3V") (layer "In2.Cu") (name "+3.3V") (hatch edge 0.508)
+  (zone (net 6) (net_name "+3V3") (layer "In2.Cu") (name "+3.3V") (hatch edge 0.508)
     (connect_pads (clearance 0.508))
     (min_thickness 0.254) (filled_areas_thickness no)
