File: BikeCam.kicad_sch (KiCad schematic)
At the start: 23 parts, among them IC1 FS312F-G, J1 USB_OTG, J2 Conn_01x02_Female, Q1 IRLZ34N, Q2 IRLZ34N, Q3 IRLML5203, Q4 IRLML5203, U1 MCP73831-2-OT, U2 LTC3531ES6-3_3

Commit message: pcb trace
Parts:
- removed IC1: FS312F-G, Package_TO_SOT_SMD:SOT-23-6, symbol FS312F-G:FS312F-G
- removed L1: 10uH, Inductor_SMD:L_1812_4532Metric, symbol Device:L
- removed U2: LTC3531ES6-3_3, Package_TO_SOT_SMD:TSOT-23-6, symbol LTC3531ES6-3_3:LTC3531ES6-3_3
- added J3: Conn_01x02_Male, Connector_PinHeader_1.00mm:PinHeader_1x02_P1.00mm_Vertical, symbol Connector:Conn_01x02_Male
- added SW1: SW_DIP_x01, Connector_PinHeader_1.00mm:PinHeader_1x02_P1.00mm_Vertical, symbol Switch:SW_DIP_x01
- added U2: AP9101CK6, Package_TO_SOT_SMD:SOT-23-6, symbol Battery_Management:AP9101CK6
- added U3: MCP1700-3302E_SOT23, Package_TO_SOT_SMD:SOT-23, symbol Regulator_Linear:MCP1700-3302E_SOT23
- C4: value 2.2uF -> 1uF
- C5: value 10uF -> 1uF
- R3: value 1k -> 2.7k
Connections:
- net +3.3V: now also U3.2 (VO)
- net GND: now also U3.1 (GND)
- net LIPO+: now also J3.2 (Pin_2)
- net LIPO-: now also J3.1 (Pin_1), U2.6 (VSS)
- net OUT+: now also SW1.2, U3.3 (VI); no longer C3.2, D2.1 (K), Q4.3 (D)
- net at C2.2, R4.1: now also U2.5 (VDD)
- net at Q2.1 (G): now also U2.1 (DO)
- net at R3.1: now also U2.2 (VM)
- net at Q1.1 (G): now also U2.3 (CO)
- new net: C3.2, D2.1 (K), Q4.3 (D), SW1.1
- no-connect marks 5 -> 4
Other:
- note added: "Voltage Regulators (LDO)"
- note removed: "Voltage Regulators (Buck-Boost)"

Commit message: pwr module debugging
Connections:
- net LIPO+: no longer J3.2 (Pin_2)
- net LIPO-: no longer J3.1 (Pin_1)
Other:
- moved on the sheet: J3
Changed lines of the file:
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@@
     (pin "2")
   )
-  (symbol (lib_id "Connector:Conn_01x02_Male") (at 121.92 186.69 180) (unit 1)
+  (symbol (lib_id "Connector:Conn_01x02_Male") (at 121.92 186.69 0) (mirror x) (unit 1)
     (in_bom yes) (on_board yes) (fields_autoplaced)
-    (property "Reference" "J3" (id 0) (at 123.19 184.1499 0)
+    (property "Reference" "J3" (id 0) (at 120.65 184.1499 0)
       (effects (font (size 1.27 1.27)) (justify right))
     )
-    (property "Value" "Conn_01x02_Male" (id 1) (at 123.19 186.6899 0)
+    (property "Value" "Conn_01x02_Male" (id 1) (at 120.65 186.6899 0)
       (effects (font (size 1.27 1.27)) (justify right))
     )

Commit message: v1
Parts:
- J2: footprint Connector_PinSocket_1.00mm:PinSocket_1x02_P1.00mm_Vertical -> Connector_PinSocket_2.00mm:PinSocket_1x02_P2.00mm_Vertical
- J3, SW1: footprint Connector_PinHeader_1.00mm:PinHeader_1x02_P1.00mm_Vertical -> Connector_PinHeader_2.00mm:PinHeader_1x02_P2.00mm_Vertical
Connections:
- net LIPO+: now also J3.1 (Pin_1)
- net LIPO-: now also J3.2 (Pin_2)
Other:
- moved on the sheet: J3
Changed lines of the file:
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@@
+    (stroke (width 0) (type default) (color 0 0 0 0))
+  )
+  (wire (pts (xy 113.03 186.69) (xy 116.84 186.69))
     (stroke (width 0) (type default) (color 0 0 0 0))
   )
@@
   )
   (wire (pts (xy 109.22 67.31) (xy 106.68 67.31))
-    (stroke (width 0) (type default) (color 0 0 0 0))
-  )
-  (wire (pts (xy 113.03 186.69) (xy 116.84 186.69))
     (stroke (width 0) (type default) (color 0 0 0 0))
   )
@@
     (pin "2")
   )
-  (symbol (lib_id "Connector:Conn_01x02_Male") (at 121.92 186.69 0) (mirror x) (unit 1)
-    (in_bom yes) (on_board yes) (fields_autoplaced)
-    (property "Reference" "J3" (id 0) (at 120.65 184.1499 0)
-      (effects (font (size 1.27 1.27)) (justify right))
-    )
-    (property "Value" "Conn_01x02_Male" (id 1) (at 120.65 186.6899 0)
-      (effects (font (size 1.27 1.27)) (justify right))
-    )
-    (property "Footprint" "Connector_PinHeader_1.00mm:PinHeader_1x02_P1.00mm_Vertical" (id 2) (at 121.92 186.69 0)
-      (effects (font (size 1.27 1.27)) hide)
-    )
-    (property "Datasheet" "~" (id 3) (at 121.92 186.69 0)
+  (symbol (lib_id "Connector:Conn_01x02_Male") (at 121.92 184.15 0) (mirror y) (unit 1)
+    (in_bom yes) (on_board yes)
+    (property "Reference" "J3" (id 0) (at 123.19 186.6901 0)
+      (effects (font (size 1.27 1.27)) (justify right))
+    )
+    (property "Value" "Conn_01x02_Male" (id 1) (at 123.19 180.34 0)
+      (effects (font (size 1.27 1.27)) (justify right))
+    )
+    (property "Footprint" "Connector_PinHeader_2.00mm:PinHeader_1x02_P2.00mm_Vertical" (id 2) (at 121.92 184.15 0)
+      (effects (font (size 1.27 1.27)) hide)
+    )
+    (property "Datasheet" "~" (id 3) (at 121.92 184.15 0)
       (effects (font (size 1.27 1.27)) hide)
     )
@@
       (effects (font (size 1.27 1.27)) (justify left))
     )
-    (property "Footprint" "Connector_PinSocket_1.00mm:PinSocket_1x02_P1.00mm_Vertical" (id 2) (at 71.12 184.15 0)
+    (property "Footprint" "Connector_PinSocket_2.00mm:PinSocket_1x02_P2.00mm_Vertical" (id 2) (at 71.12 184.15 0)
       (effects (font (size 1.27 1.27)) hide)
     )
@@
     (property "Reference" "SW1" (id 0) (at 191.77 50.8 0))
     (property "Value" "SW_DIP_x01" (id 1) (at 191.77 53.34 0))
-    (property "Footprint" "Connector_PinHeader_1.00mm:PinHeader_1x02_P1.00mm_Vertical" (id 2) (at 184.15 58.42 0)
+    (property "Footprint" "Connector_PinHeader_2.00mm:PinHeader_1x02_P2.00mm_Vertical" (id 2) (at 184.15 58.42 0)
       (effects (font (size 1.27 1.27)) hide)
     )
@@
     )
     (path "/3f651b51-c339-4160-a87b-1cdb926631ea"
-      (reference "J2") (unit 1) (value "Conn_01x02_Female") (footprint "Connector_PinSocket_1.00mm:PinSocket_1x02_P1.00mm_Vertical")
+      (reference "J2") (unit 1) (value "Conn_01x02_Female") (footprint "Connector_PinSocket_2.00mm:PinSocket_1x02_P2.00mm_Vertical")
     )
     (path "/1b0fdc69-3f2d-4e8c-a8f4-606e3a3e3f53"
-      (reference "J3") (unit 1) (value "Conn_01x02_Male") (footprint "Connector_PinHeader_1.00mm:PinHeader_1x02_P1.00mm_Vertical")
+      (reference "J3") (unit 1) (value "Conn_01x02_Male") (footprint "Connector_PinHeader_2.00mm:PinHeader_1x02_P2.00mm_Vertical")
     )
     (path "/df922417-c436-4308-ade5-eb9718caada6"
@@
     )
     (path "/6d1a7f34-63c4-483b-aa39-b67b33e4babb"
-      (reference "SW1") (unit 1) (value "SW_DIP_x01") (footprint "Connector_PinHeader_1.00mm:PinHeader_1x02_P1.00mm_Vertical")
+      (reference "SW1") (unit 1) (value "SW_DIP_x01") (footprint "Connector_PinHeader_2.00mm:PinHeader_1x02_P2.00mm_Vertical")
     )
     (path "/90b76ee2-5cd6-4abc-a51e-e2b414b967d0"

Commit message: error debug
Connections:
- net +3.3V renamed +3V3
Changed lines of the file:
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@@
   (junction (at 160.02 50.8) (diameter 0) (color 0 0 0 0)
   )
-  (no_connect (at 24.13 187.96))
-  (no_connect (at 34.29 180.34))
-  (no_connect (at 34.29 182.88))
-  (no_connect (at 34.29 177.8))
+  (no_connect (at 36.83 180.34))
+  (no_connect (at 24.13 190.5))
+  (no_connect (at 36.83 182.88))
+  (no_connect (at 36.83 177.8))
   (wire (pts (xy 160.02 41.91) (xy 172.72 41.91))
     (stroke (width 0) (type default) (color 0 0 0 0))
@@
     (stroke (width 0) (type default) (color 0 0 0 0))
   )
-  (wire (pts (xy 63.5 184.15) (xy 66.04 184.15))
-    (stroke (width 0) (type default) (color 0 0 0 0))
-  )
-  (wire (pts (xy 248.92 45.72) (xy 251.46 45.72))
+  (wire (pts (xy 60.96 184.15) (xy 66.04 184.15))
+    (stroke (width 0) (type default) (color 0 0 0 0))
+  )
+  (wire (pts (xy 248.92 45.72) (xy 255.27 45.72))
     (stroke (width 0) (type default) (color 0 0 0 0))
   )
@@
     (stroke (width 0) (type default) (color 0 0 0 0))
   )
+  (wire (pts (xy 34.29 177.8) (xy 36.83 177.8))
+    (stroke (width 0) (type default) (color 0 0 0 0))
+  )
   (wire (pts (xy 118.11 74.93) (xy 121.92 74.93))
     (stroke (width 0) (type default) (color 0 0 0 0))
@@
     (stroke (width 0) (type default) (color 0 0 0 0))
   )
+  (wire (pts (xy 34.29 180.34) (xy 36.83 180.34))
+    (stroke (width 0) (type default) (color 0 0 0 0))
+  )
   (wire (pts (xy 87.63 71.12) (xy 87.63 74.93))
     (stroke (width 0) (type default) (color 0 0 0 0))
@@
     (stroke (width 0) (type default) (color 0 0 0 0))
   )
+  (wire (pts (xy 34.29 182.88) (xy 36.83 182.88))
+    (stroke (width 0) (type default) (color 0 0 0 0))
+  )
   (wire (pts (xy 172.72 66.04) (xy 172.72 67.31))
     (stroke (width 0) (type default) (color 0 0 0 0))
@@
   )
   (wire (pts (xy 53.34 48.26) (xy 53.34 55.88))
+    (stroke (width 0) (type default) (color 0 0 0 0))
+  )
+  (wire (pts (xy 24.13 187.96) (xy 24.13 190.5))
     (stroke (width 0) (type default) (color 0 0 0 0))
   )
@@
     )
   )
-  (global_label "+3.3V" (shape input) (at 63.5 184.15 180) (fields_autoplaced)
-    (effects (font (size 1.27 1.27)) (justify right))
-    (property "Intersheet References" "${INTERSHEET_REFS}" (id 0) (at 55.4021 184.2294 0)
-      (effects (font (size 1.27 1.27)) (justify right) hide)
-    )
-  )
   (global_label "LIPO+" (shape input) (at 113.03 184.15 180) (fields_autoplaced)
     (effects (font (size 1.27 1.27)) (justify right))
@@
     )
   )
-  (global_label "+3.3V" (shape input) (at 251.46 45.72 0) (fields_autoplaced)
-    (effects (font (size 1.27 1.27)) (justify left))
-    (property "Intersheet References" "${INTERSHEET_REFS}" (id 0) (at 259.5579 45.6406 0)
-      (effects (font (size 1.27 1.27)) (justify left) hide)
-    )
-  )
   (global_label "0V" (shape input) (at 30.48 74.93 180) (fields_autoplaced)
     (effects (font (size 1.27 1.27)) (justify right))
@@
     (pin "2")
   )
+  (symbol (lib_id "power:+3V3") (at 255.27 45.72 0) (unit 1)
+    (in_bom yes) (on_board yes) (fields_autoplaced)
+    (property "Reference" "#PWR06" (id 0) (at 255.27 49.53 0)
+      (effects (font (size 1.27 1.27)) hide)
+    )
+    (property "Value" "+3V3" (id 1) (at 255.27 40.64 0))
+    (property "Footprint" "" (id 2) (at 255.27 45.72 0)
+      (effects (font (size 1.27 1.27)) hide)
+    )
+    (property "Datasheet" "" (id 3) (at 255.27 45.72 0)
+      (effects (font (size 1.27 1.27)) hide)
+    )
+    (pin "1")
+  )
   (symbol (lib_id "power:PWR_FLAG") (at 36.83 172.72 0) (unit 1)
     (in_bom yes) (on_board yes)
@@
   (symbol (lib_id "power:GND") (at 229.87 53.34 0) (mirror y) (unit 1)
     (in_bom yes) (on_board yes) (fields_autoplaced)
-    (property "Reference" "#PWR03" (id 0) (at 229.87 59.69 0)
+    (property "Reference" "#PWR04" (id 0) (at 229.87 59.69 0)
       (effects (font (size 1.27 1.27)) hide)
     )
@@
   (symbol (lib_id "power:GND") (at 68.58 77.47 0) (mirror y) (unit 1)
     (in_bom yes) (on_board yes) (fields_autoplaced)
-    (property "Reference" "#PWR01" (id 0) (at 68.58 83.82 0)
+    (property "Reference" "#PWR02" (id 0) (at 68.58 83.82 0)
       (effects (font (size 1.27 1.27)) hide)
     )
@@
     (pin "2")
   )
+  (symbol (lib_id "power:+3V3") (at 60.96 184.15 0) (unit 1)
+    (in_bom yes) (on_board yes) (fields_autoplaced)
+    (property "Reference" "#PWR01" (id 0) (at 60.96 187.96 0)
+      (effects (font (size 1.27 1.27)) hide)
+    )
+    (property "Value" "+3V3" (id 1) (at 60.96 179.07 0))
+    (property "Footprint" "" (id 2) (at 60.96 184.15 0)
+      (effects (font (size 1.27 1.27)) hide)
+    )
+    (property "Datasheet" "" (id 3) (at 60.96 184.15 0)
+      (effects (font (size 1.27 1.27)) hide)
+    )
+    (pin "1")
+  )
   (symbol (lib_id "Transistor_FET:IRLZ34N") (at 96.52 72.39 270) (unit 1)
     (in_bom yes) (on_board yes) (fields_autoplaced)
@@
   (symbol (lib_id "power:GND") (at 248.92 53.34 0) (mirror y) (unit 1)
     (in_bom yes) (on_board yes) (fields_autoplaced)
-    (property "Reference" "#PWR04" (id 0) (at 248.92 59.69 0)
+    (property "Reference" "#PWR05" (id 0) (at 248.92 59.69 0)
       (effects (font (size 1.27 1.27)) hide)
     )
@@
   (symbol (lib_id "power:GND") (at 172.72 68.58 0) (mirror y) (unit 1)
     (in_bom yes) (on_board yes) (fields_autoplaced)
-    (property "Reference" "#PWR02" (id 0) (at 172.72 74.93 0)
+    (property "Reference" "#PWR03" (id 0) (at 172.72 74.93 0)
       (effects (font (size 1.27 1.27)) hide)
     )
@@
       (reference "#FLG05") (unit 1) (value "PWR_FLAG") (footprint "")
     )
+    (path "/cf871db5-77ca-41bf-93a8-99f564c1793a"
+      (reference "#PWR01") (unit 1) (value "+3V3") (footprint "")
+    )
     (path "/70995274-7314-4c3f-8138-677f4afc9311"
-      (reference "#PWR01") (unit 1) (value "GND") (footprint "")
+      (reference "#PWR02") (unit 1) (value "GND") (footprint "")
     )
     (path "/f59ee7f6-6993-4c33-8bd2-12b0e6695513"
-      (reference "#PWR02") (unit 1) (value "GND") (footprint "")
+      (reference "#PWR03") (unit 1) (value "GND") (footprint "")
     )
     (path "/4d7dceab-0373-46c3-a89a-47505835f6d7"
-      (reference "#PWR03") (unit 1) (value "GND") (footprint "")
+      (reference "#PWR04") (unit 1) (value "GND") (footprint "")
     )
     (path "/edb571f5-8f53-4e77-9c3c-121afa122d2b"
-      (reference "#PWR04") (unit 1) (value "GND") (footprint "")
+      (reference "#PWR05") (unit 1) (value "GND") (footprint "")
+    )
+    (path "/2195ac39-3cd5-4eef-b9fb-ee5b4e72c7bc"
+      (reference "#PWR06") (unit 1) (value "+3V3") (footprint "")
     )
     (path "/46fb08e3-6a0c-4eeb-a85e-163548014295"
